File: ratt.kicad_sch (KiCad schematic)
At the start: 33 parts, among them J1 Conn_01x04_Male, J2 Conn_01x04_Male, Q1 2N5457, U1 LM308N

Commit message: updated rotation of pots.
Parts:
- added J3, J4: Conn_01x01_Male, Connector_PinSocket_2.54mm:PinSocket_1x01_P2.54mm_Vertical, symbol Connector:Conn_01x01_Male
Connections:
- net at C8.1, R11.2, R8.2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: now also RV3.3; no longer RV3.1
- net at C2.1, C8.2, U1.6: now also RV3.1; no longer RV3.3
- net at C10.1, RV2.2: now also RV2.1; no longer RV2.3
- net at R8.1: now also RV2.3; no longer RV2.1
Other:
- moved on the sheet: RV3
Changed lines of the file:
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@@
     (pin "2")
   )
-  (symbol (lib_id "Device:R_Potentiometer") (at 158.242 165.735 90) (mirror x) (unit 1)
+  (symbol (lib_id "Device:R_Potentiometer") (at 158.242 165.735 270) (unit 1)
     (in_bom yes) (on_board yes)
     (property "Reference" "RV3" (id 0) (at 158.242 160.528 90))
@@
     (pin "1")
   )
+  (symbol (lib_id "Connector:Conn_01x01_Male") (at 39.624 130.048 0) (unit 1)
+    (in_bom yes) (on_board yes) (fields_autoplaced)
+    (property "Reference" "J4" (id 0) (at 40.259 124.714 0))
+    (property "Value" "Conn_01x01_Male" (id 1) (at 40.259 127.254 0))
+    (property "Footprint" "Connector_PinSocket_2.54mm:PinSocket_1x01_P2.54mm_Vertical" (id 2) (at 39.624 130.048 0)
+      (effects (font (size 1.27 1.27)) hide)
+    )
+    (property "Datasheet" "~" (id 3) (at 39.624 130.048 0)
+      (effects (font (size 1.27 1.27)) hide)
+    )
+    (pin "1")
+  )
   (symbol (lib_id "power:GND") (at 131.826 145.415 0) (unit 1)
     (in_bom yes) (on_board yes) (fields_autoplaced)
@@
     (pin "2")
   )
-  (symbol (lib_id "Device:R_Potentiometer") (at 114.046 162.814 0) (unit 1)
-    (in_bom yes) (on_board yes) (fields_autoplaced)
-    (property "Reference" "RV2" (id 0) (at 111.506 161.5439 0)
-      (effects (font (size 1.27 1.27)) (justify right))
-    )
-    (property "Value" "B1k" (id 1) (at 111.506 164.0839 0)
+  (symbol (lib_id "Device:R_Potentiometer") (at 114.046 162.814 0) (mirror x) (unit 1)
+    (in_bom yes) (on_board yes) (fields_autoplaced)
+    (property "Reference" "RV2" (id 0) (at 111.76 161.5439 0)
+      (effects (font (size 1.27 1.27)) (justify right))
+    )
+    (property "Value" "B1k" (id 1) (at 111.76 164.0839 0)
       (effects (font (size 1.27 1.27)) (justify right))
     )
@@
     (pin "3")
   )
+  (symbol (lib_id "Connector:Conn_01x01_Male") (at 39.624 121.666 0) (unit 1)
+    (in_bom yes) (on_board yes) (fields_autoplaced)
+    (property "Reference" "J3" (id 0) (at 40.259 116.332 0))
+    (property "Value" "Conn_01x01_Male" (id 1) (at 40.259 118.872 0))
+    (property "Footprint" "Connector_PinSocket_2.54mm:PinSocket_1x01_P2.54mm_Vertical" (id 2) (at 39.624 121.666 0)
+      (effects (font (size 1.27 1.27)) hide)
+    )
+    (property "Datasheet" "~" (id 3) (at 39.624 121.666 0)
+      (effects (font (size 1.27 1.27)) hide)
+    )
+    (pin "1")
+  )
   (symbol (lib_id "Device:C_Polarized_US") (at 134.366 174.879 0) (unit 1)
     (in_bom yes) (on_board yes)
@@
       (reference "J2") (unit 1) (value "Conn_01x04_Male") (footprint "Connector_PinHeader_2.54mm:PinHeader_1x04_P2.54mm_Vertical")
     )
+    (path "/f1403e7f-5f08-4c8d-82fe-41f6ffce7562"
+      (reference "J3") (unit 1) (value "Conn_01x01_Male") (footprint "Connector_PinSocket_2.54mm:PinSocket_1x01_P2.54mm_Vertical")
+    )
+    (path "/a47ca0f0-1272-4c92-81c6-223879630a80"
+      (reference "J4") (unit 1) (value "Conn_01x01_Male") (footprint "Connector_PinSocket_2.54mm:PinSocket_1x01_P2.54mm_Vertical")
+    )
     (path "/f003d1d6-a76e-4138-b0ce-e137e978b103"
